File: vermona-regent-1010.kicad_pcb (KiCad board)
At the start: 2 copper layers, 62 parts, among them J1 Input, Q1 КТ3102Б, Q10 КТ814Г, Q11 КТ808, Q12 КТ808, Q2 КТ3102Б, Q3 КТ3102Б, Q4 КТ815Г, Q5 КТ814Г, Q6 КТ3102Б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

Commit message: Finish routing amp
Parts:
- added J2: -40V, Connector_PinHeader_2.54mm:PinHeader_1x02_P2.54mm_Vertical, F.Cu at (179.1, 100.3)
- added J3: +40V, Connector_PinHeader_2.54mm:PinHeader_1x02_P2.54mm_Vertical, F.Cu at (179.1, 94.0)
- moved R8 337.2 mm to (80.0, 73.7), turned to 270 degrees
- moved C12 328.6 mm to (97.8, 91.4), turned to 180 degrees
- moved R15 319.1 mm to (109.2, 124.5), turned to 90 degrees
- moved D6 316.9 mm to (92.7, 124.5), turned to 90 degrees
- moved C9 315.4 mm to (102.9, 100.3), turned to 90 degrees
- moved Q6 313.0 mm to (95.2, 99.1)
- moved Q7 311.7 mm to (125.7, 95.2), turned to 180 degrees
- moved RV2 302.1 mm to (87.6, 101.6), turned to 90 degrees
- moved R12 287.2 mm to (120.7, 88.9), turned to 90 degrees
- moved Q12 284.8 mm to (143.5, 102.9)
- moved Q11 284.3 mm to (143.5, 88.9)
- moved Q9 282.8 mm to (137.2, 88.9), turned to 270 degrees
- moved R9 281.1 mm to (90.2, 73.7), turned to 270 degrees
- moved R13 279.7 mm to (104.1, 124.5), turned to 90 degrees
- moved Q8 278.6 mm to (125.1, 108.6), turned to 180 degrees
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Routing:
- net 40V: track 21.6 -> 188.5 mm
- net -40V: track 0.00 -> 161.7 mm
- net Net-(C12-Pad2): track 0.00 -> 127.6 mm
- net Net-(C14-Pad2): track 0.00 -> 114.9 mm
- net Net-(C12-Pad1): track 0.00 -> 84.3 mm
- net GND: track 0.00 -> 66.3 mm
- net Net-(C6-Pad2): track 0.00 -> 63.5 mm
- net Net-(C7-Pad1): track 0.00 -> 59.4 mm
- net Net-(Q10-Pad2): track 0.00 -> 51.7 mm
- net Net-(Q11-Pad2): track 0.00 -> 41.3 mm
- net Net-(Q1-Pad2): track 5.08 -> 40.8 mm
- net Net-(C15-Pad2): track 0.00 -> 31.7 mm
- net Net-(D6-Pad2): track 0.00 -> 31.2 mm
- net Net-(F1-Pad2): track 0.00 -> 28.8 mm
- net Net-(C9-Pad2): track 0.00 -> 27.3 mm
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